File: aux-io.brd (EAGLE design)
At the start: 50 x 80 mm, 123 parts, among them X4 MPT0.5/8-2.54, X5 MPT0.5/8-2.54, X6 X3815-10, X7 MPT0.5/8-2.54, Y1 PTH2.6-5.5SQ, Y2 PTH2.6-5.5SQ, Y3 PTH2.6-5.5SQ, Y4 PTH2.6-5.5SQ

Commit message: routed
Parts:
- added DRILEGEND: (no value), drilegend:DRILEGEND
- added U$1: DAFUG, omat:DAFUG
- Y1, Y2, Y3, Y4: value PTH2.6-5.5SQ -> PTH; device EKE:PTH-2.6-5.5SQ -> omat:PTH-3.2-6DIA
- moved C2 10.0 mm to (39.2, 17.8)
- moved C19 7.23 mm to (27.8, 41.4)
- moved C20 5.90 mm to (33.0, 46.1), flipped to the top, turned to 90 degrees
- moved C22 5.75 mm to (22.0, 37.2), turned to 180 degrees
- moved R32 4.93 mm to (35.1, 42.8)
- moved C14 3.52 mm to (33.6, 32.0)
- moved C25 3.52 mm to (28.6, 32.0)
- moved R27 3.52 mm to (34.6, 27.0)
- moved R28 3.52 mm to (35.6, 32.0)
- moved R29 3.52 mm to (29.6, 27.0)
- moved R39 3.52 mm to (30.6, 32.0)
- moved C16 3.40 mm to (19.2, 47.0), flipped to the top, turned to 180 degrees
- moved C1 3.04 mm to (36.5, 11.0), flipped to the top, turned to 0 degrees
- moved C21 2.38 mm to (22.0, 41.4), turned to 180 degrees
- moved R31 1.77 mm to (13.2, 39.2)
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Connections:
- net MOTOR2_H1: now also D1.25; no longer D1.24
- net MOTOR2_H2: now also D1.24; no longer D1.25
Routing:
- net GND: track 0.00 -> 261.3 mm, vias 0 -> 78
- net +12V: track 0.00 -> 207.6 mm, vias 0 -> 6
- net +3V3: track 0.00 -> 149.2 mm, vias 0 -> 7
- net MOTOR2A: track 0.00 -> 38.2 mm
- net MOTOR1A: track 0.00 -> 37.2 mm
- net MOTOR1_L1: track 0.00 -> 33.6 mm
- net RESETL: track 0.00 -> 32.9 mm, vias 0 -> 2
- net INPUT2: track 0.00 -> 32.7 mm
- net MOTOR1_L2: track 0.00 -> 31.8 mm
- net INPUT1: track 0.00 -> 30.2 mm
- net ACCLINKTXE: track 0.00 -> 29.8 mm, vias 0 -> 2
- net SWCLK_CPU: track 0.00 -> 27.8 mm, vias 0 -> 2
- net ACCLINKTX: track 0.00 -> 27.5 mm, vias 0 -> 2
- net USART6RX: track 0.00 -> 27.5 mm, vias 0 -> 2
- net MOTOR1_H2: track 0.00 -> 27.1 mm, vias 0 -> 2
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- added copper zone on layer 1, net GND
- added copper zone on layer 16, net GND
Other:
- board text added: "(C) 2018 KIMMOLI"
- board text added: "+"
- board text added: "-"
- board text added: "01-16"
- board text added: "01-20"
- board text added: "LAYER-STACK"
- board text added: "TELAKONE AUX IO"
