File: aux-io.sch (EAGLE design)
At the start: 123 parts, among them X4 MPT0.5/8-2.54, X5 MPT0.5/8-2.54, X6 X3815-10, X7 MPT0.5/8-2.54, Y1 PTH2.6-5.5SQ, Y2 PTH2.6-5.5SQ, Y3 PTH2.6-5.5SQ, Y4 PTH2.6-5.5SQ

Commit message: routed
Parts:
- added U$1: DAFUG, omat:DAFUG
- Y1, Y2, Y3, Y4: value PTH2.6-5.5SQ -> PTH; device EKE:PTH2.6-5.5SQ -> omat:PTH
Connections:
- net MOTOR2_H1: now also D1G$2.PC5; no longer D1G$2.PC4
- net MOTOR2_H2: now also D1G$2.PC4; no longer D1G$2.PC5
Changed lines of the file:
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@@
 <part name="GND30" library="EKE" deviceset="GND" device=""/>
 <part name="+3V5" library="EKE" deviceset="+3V3" device=""/>
-<part name="Y1" library="EKE" deviceset="PTH" device="2.6-5.5SQ"/>
-<part name="Y2" library="EKE" deviceset="PTH" device="2.6-5.5SQ"/>
-<part name="Y3" library="EKE" deviceset="PTH" device="2.6-5.5SQ"/>
-<part name="Y4" library="EKE" deviceset="PTH" device="2.6-5.5SQ"/>
+<part name="Y1" library="omat" deviceset="PTH" device=""/>
+<part name="Y2" library="omat" deviceset="PTH" device=""/>
+<part name="Y3" library="omat" deviceset="PTH" device=""/>
+<part name="Y4" library="omat" deviceset="PTH" device=""/>
 <part name="GND77" library="EKE" deviceset="GND" device=""/>
 <part name="G1" library="omat_ic_2" deviceset="XTAL_3225_SMD" device="" value="25MHz"/>
@@
 <part name="R41" library="passiivit" deviceset="RES" device="0603"/>
 <part name="GND6" library="EKE" deviceset="GND" device=""/>
+<part name="U$1" library="omat" deviceset="DAFUG" device=""/>
 </parts>
 <sheets>
@@
 <attribute name="VALUE" x="281.94" y="165.1" size="1.778" layer="96"/>
 </instance>
+<instance part="U$1" gate="G$1" x="289.56" y="25.4" smashed="yes"/>
 </instances>
 <busses>
@@
 <label x="139.7" y="175.26" size="1.778" layer="95"/>
 <pinref part="D1" gate="G$2" pin="PA1"/>
-</segment>
-</net>
-<net name="MOTOR2_H1" class="0">
-<segment>
-<wire x1="213.36" y1="165.1" x2="241.3" y2="165.1" width="0.1524" layer="91"/>
-<label x="220.98" y="165.1" size="1.778" layer="95"/>
-<pinref part="D1" gate="G$2" pin="PC4"/>
-</segment>
-</net>
-<net name="MOTOR2_H2" class="0">
-<segment>
-<wire x1="213.36" y1="162.56" x2="241.3" y2="162.56" width="0.1524" layer="91"/>
-<label x="220.98" y="162.56" size="1.778" layer="95"/>
-<pinref part="D1" gate="G$2" pin="PC5"/>
 </segment>
 </net>
@@
 </segment>
 </net>
+<net name="MOTOR2_H2" class="0">
+<segment>
+<pinref part="D1" gate="G$2" pin="PC4"/>
+<wire x1="213.36" y1="165.1" x2="241.3" y2="165.1" width="0.1524" layer="91"/>
+<label x="220.98" y="165.1" size="1.778" layer="95"/>
+</segment>
+</net>
+<net name="MOTOR2_H1" class="0">
+<segment>
+<pinref part="D1" gate="G$2" pin="PC5"/>
+<wire x1="213.36" y1="162.56" x2="241.3" y2="162.56" width="0.1524" layer="91"/>
+<label x="220.98" y="162.56" size="1.778" layer="95"/>
+</segment>
+</net>
